File: Schematic/Quadriscope.kicad_sch (KiCad schematic)
At the start: 65 parts, among them IC101 LD1117-3.3V-SOT223, J101 IN_1, J102 THRU_1, J103 IN_2, J104 THRU_2, J105 IN_3, J106 THRU_3, J107 IN_4, J108 THRU_4, J109 Conn_02x05_Odd_Even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

Commit message: new board file, interrupt stuff
Parts:
- R119: value 51k -> 89k
Connections:
- net +3.3V: no longer C101.1, C112.1, L101.2, U102.2 (~{RST/PD}), U102.30 (AVDD), U102.34 (DVDD), U102.9 (AVDD)
- net +5V: now also C101.1, C112.1, L101.2, R119.2, U102.2 (~{RST/PD}), U102.30 (AVDD), U102.34 (DVDD), U102.9 (AVDD)
- net ADC_CS: now also U101.33 (MTDO/GPIO40/CLK_OUT2); no longer U101.18 (GPIO10/TOUCH10/ADC1_CH9/FSPICS0/FSPIIO4/SUBSPICS0)
- net ADC_MOSI: now also U101.32 (MTCK/GPIO39/CLK_OUT3/SUBSPICS1); no longer U101.19 (GPIO11/TOUCH11/ADC2_CH0/FSPID/FSPIIO5/SUBSPID)
- net ENCB_B: now also U101.34 (MTDI/GPIO41/CLK_OUT1); no longer U101.17 (GPIO9/TOUCH9/ADC1_CH8/FSPIHD/SUBSPIHD)
- net ENCB_L: now also U101.9 (GPIO16/U0CTS/ADC2_CH5/XTAL_32K_N); no longer U101.7 (GPIO7/TOUCH7/ADC1_CH6)
- net ENCB_R: now also U101.35 (MTMS/GPIO42); no longer U101.12 (GPIO8/TOUCH8/ADC1_CH7/SUBSPICS1)
- net at C111.2, L101.1, U103.6 (SW): no longer R119.1
- net at R120.1, U103.3 (FB): now also R119.1; no longer R119.2
Other:
- note added: "5v Buck Converter"
- note removed: "3.3v Buck Converter"
- title: Eurorack 4-Ch Oscilloscope -> Quadriscope
- moved on the sheet: C112, R119
